File: hw/baloon.sch (KiCad schematic (older format))
At the start: 33 parts, among them J1 SOLAR, J2 DEBUG, J3 SWO, J4 ANT, J5 ANT, Q3 DMP2035, U1 STM32F030C8Tx, U2 Si7020-A20, U3 MS5607-02BA, U4 RFM95W-868S2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

Commit message: Final board
Parts:
- removed C5: 1u, Capacitor_SMD:C_0603_1608Metric, symbol Device:C
- added JP1: backup, Jumper:SolderJumper-3_P1.3mm_Open_RoundedPad1.0x1.5mm, symbol Jumper:SolderJumper_3_Open
- J2: footprint Connector_PinHeader_1.27mm:PinHeader_1x03_P1.27mm_Vertical -> Connector_PinSocket_1.00mm:PinSocket_1x03_P1.00mm_Vertical_SMD_Pin1Left
Connections:
- wire segments 179 -> 178
Other:
- moved on the sheet: C14, C6
Changed lines of the file:
@@
 Sheet 1 2
 Title "Deadbadger PicoBalloon Challenge probe"
-Date "2020-01-10"
-Rev "0.1"
+Date "2020-01-13"
+Rev "0.2"
 Comp "Deadbadger.cz"
 Comment1 ""
@@
 SWDIO
 Wire Wire Line
-	1700 6050 2150 6050
-Wire Wire Line
-	1700 6150 2150 6150
-Wire Wire Line
-	1700 6250 2150 6250
-Text Label 1700 6050 0    50   ~ 0
-SCK
-Text Label 1700 6150 0    50   ~ 0
-MISO
-Text Label 1700 6250 0    50   ~ 0
-MOSI
-Wire Wire Line
 	2150 5350 1050 5350
 Text Label 850  5350 0    50   ~ 0
@@
 F 0 "J2" H 5468 6975 50  0000 C CNN
 F 1 "DEBUG" H 5468 7066 50  0000 C CNN
-F 2 "Connector_PinHeader_1.27mm:PinHeader_1x03_P1.27mm_Vertical" H 5550 7300 50  0001 C CNN
+F 2 "Connector_PinSocket_1.00mm:PinSocket_1x03_P1.00mm_Vertical_SMD_Pin1Left" H 5550 7300 50  0001 C CNN
 F 3 "~" H 5550 7300 50  0001 C CNN
 	1    5550 7300
@@
 $EndComp
 $Comp
-L Device:C C5
-U 1 1 5E2C7007
-P 1600 7300
-F 0 "C5" H 1715 7346 50  0000 L CNN
-F 1 "1u" H 1715 7255 50  0000 L CNN
-F 2 "Capacitor_SMD:C_0603_1608Metric" H 1638 7150 50  0001 C CNN
-F 3 "~" H 1600 7300 50  0001 C CNN
-	1    1600 7300
-	1    0    0    -1
-$EndComp
-$Comp
 L Device:C C6
 U 1 1 5E2C735A
-P 2050 7300
-F 0 "C6" H 2165 7346 50  0000 L CNN
-F 1 "1u" H 2165 7255 50  0000 L CNN
-F 2 "Capacitor_SMD:C_0603_1608Metric" H 2088 7150 50  0001 C CNN
-F 3 "~" H 2050 7300 50  0001 C CNN
-	1    2050 7300
+P 1650 7300
+F 0 "C6" H 1765 7346 50  0000 L CNN
+F 1 "1u" H 1765 7255 50  0000 L CNN
+F 2 "Capacitor_SMD:C_0603_1608Metric" H 1688 7150 50  0001 C CNN
+F 3 "~" H 1650 7300 50  0001 C CNN
+	1    1650 7300
 	1    0    0    -1
 $EndComp
@@
 	700  7150 700  7100
 Wire Wire Line
-	2050 7100 2050 7150
+	1650 7100 1650 7150
 Wire Wire Line
 	700  7450 700  7500
 Wire Wire Line
-	2050 7500 2050 7450
-Wire Wire Line
-	1600 7500 1600 7450
-Connection ~ 1600 7500
-Wire Wire Line
-	1600 7500 2050 7500
+	1650 7500 1650 7450
 Wire Wire Line
 	1150 7500 1150 7450
 Connection ~ 1150 7500
 Wire Wire Line
-	1150 7500 1400 7500
-Wire Wire Line
 	1150 7150 1150 7100
 Connection ~ 1150 7100
-Wire Wire Line
-	1150 7100 1400 7100
-Wire Wire Line
-	1600 7150 1600 7100
-Connection ~ 1600 7100
-Wire Wire Line
-	1600 7100 2050 7100
 $Comp
 L power:+3V3 #PWR0127
 U 1 1 5E2FF356
-P 1400 7050
-F 0 "#PWR0127" H 1400 6900 50  0001 C CNN
-F 1 "+3V3" H 1415 7223 50  0000 C CNN
-F 2 "" H 1400 7050 50  0001 C CNN
-F 3 "" H 1400 7050 50  0001 C CNN
-	1    1400 7050
+P 1150 7050
+F 0 "#PWR0127" H 1150 6900 50  0001 C CNN
+F 1 "+3V3" H 1165 7223 50  0000 C CNN
+F 2 "" H 1150 7050 50  0001 C CNN
+F 3 "" H 1150 7050 50  0001 C CNN
+	1    1150 7050
 	1    0    0    -1
 $EndComp
@@
 L Device:C C14
 U 1 1 5E3A0AFF
-P 9600 1600
-F 0 "C14" V 9348 1600 50  0000 C CNN
-F 1 "100n" V 9439 1600 50  0000 C CNN
-F 2 "Capacitor_SMD:C_0603_1608Metric" H 9638 1450 50  0001 C CNN
-F 3 "~" H 9600 1600 50  0001 C CNN
-	1    9600 1600
-	0    1    1    0
-$EndComp
-Wire Wire Line
-	9450 1600 9400 1600
-Connection ~ 9400 1600
-Wire Wire Line
-	9400 1600 9400 1900
+P 10650 1800
+F 0 "C14" V 10398 1800 50  0000 C CNN
+F 1 "100n" V 10489 1800 50  0000 C CNN
+F 2 "Capacitor_SMD:C_0603_1608Metric" H 10688 1650 50  0001 C CNN
+F 3 "~" H 10650 1800 50  0001 C CNN
+	1    10650 1800
+	0    1    1    0
+$EndComp
 $Comp
 L power:GND #PWR0131
 U 1 1 5E3A83CF
-P 9800 1600
-F 0 "#PWR0131" H 9800 1350 50  0001 C CNN
-F 1 "GND" V 9805 1472 50  0000 R CNN
-F 2 "" H 9800 1600 50  0001 C CNN
-F 3 "" H 9800 1600 50  0001 C CNN
-	1    9800 1600
+P 10850 1800
+F 0 "#PWR0131" H 10850 1550 50  0001 C CNN
+F 1 "GND" V 10855 1672 50  0000 R CNN
+F 2 "" H 10850 1800 50  0001 C CNN
+F 3 "" H 10850 1800 50  0001 C CNN
+	1    10850 1800
 	0    -1   -1   0
 $EndComp
 Wire Wire Line
-	9800 1600 9750 1600
+	10850 1800 10800 1800
 Text Notes 10650 3800 0    50   ~ 0
 Radio\n868MHz LoRa
@@
 ~POWER_OFF
 Wire Wire Line
-	3800 5450 3350 5450
-Text Label 3350 5450 0    50   ~ 0
+	3800 5150 3350 5150
+Text Label 3350 5150 0    50   ~ 0
 ~POWER_OFF
 Wire Wire Line
-	3800 5250 3350 5250
-Text Label 3500 5150 0    50   ~ 0
+	3800 5950 3350 5950
+Text Label 3500 5850 0    50   ~ 0
 RFM_IO1
-Text Label 3500 5250 0    50   ~ 0
+Text Label 3500 5950 0    50   ~ 0
 RFM_IO0
 Wire Wire Line
-	3800 5150 3350 5150
-Wire Wire Line
-	1700 5850 2150 5850
-Text Label 1700 5850 0    50   ~ 0
+	3800 5850 3350 5850
+Wire Wire Line
+	1700 4750 2150 4750
+Text Label 1700 4750 0    50   ~ 0
 RFM_CS
 Wire Wire Line
-	1700 5750 2150 5750
-Text Label 1700 5750 0    50   ~ 0
+	1700 4850 2150 4850
+Text Label 1700 4850 0    50   ~ 0
 RFM_RESET
 Wire Wire Line
@@
 NoConn ~ 2150 4550
 NoConn ~ 2150 5050
-NoConn ~ 2150 5150
 NoConn ~ 2150 5250
 NoConn ~ 2150 5550
-NoConn ~ 3350 5850
-NoConn ~ 3350 5950
+NoConn ~ 2150 6150
+NoConn ~ 2150 6250
 NoConn ~ 3350 6250
 $Comp
@@
 L power:+BATT #PWR0108
 U 1 1 5E539416
-P 9400 1450
-F 0 "#PWR0108" H 9400 1300 50  0001 C CNN
-F 1 "+BATT" H 9415 1623 50  0000 C CNN
-F 2 "" H 9400 1450 50  0001 C CNN
-F 3 "" H 9400 1450 50  0001 C CNN
-	1    9400 1450
-	1    0    0    -1
-$EndComp
-Wire Wire Line
-	9400 1450 9400 1600
+P 9400 1550
+F 0 "#PWR0108" H 9400 1400 50  0001 C CNN
+F 1 "+BATT" H 9415 1723 50  0000 C CNN
+F 2 "" H 9400 1550 50  0001 C CNN
+F 3 "" H 9400 1550 50  0001 C CNN
+	1    9400 1550
+	1    0    0    -1
+$EndComp
 Wire Wire Line
 	9200 800  9550 800
 Wire Wire Line
-	3350 5350 3800 5350
-Text Label 3350 5350 0    50   ~ 0
+	1700 5150 2150 5150
+Text Label 1700 5150 0    50   ~ 0
 ~GPS_POWER
 NoConn ~ 2150 5950
 NoConn ~ 2150 5650
 NoConn ~ 3350 5550
-NoConn ~ 2150 4850
+NoConn ~ 2150 6050
 NoConn ~ 2150 4950
 $Comp
@@
 Text Label 10700 1200 0    50   ~ 0
 ~GPS_POWER
-NoConn ~ 2150 4750
+NoConn ~ 2150 5850
 Wire Wire Line
 	10200 800  10200 850
@@
 L power:GND #PWR0128
 U 1 1 5E306464
-P 1400 7550
-F 0 "#PWR0128" H 1400 7300 50  0001 C CNN
-F 1 "GND" H 1405 7377 50  0000 C CNN
-F 2 "" H 1400 7550 50  0001 C CNN
-F 3 "" H 1400 7550 50  0001 C CNN
-	1    1400 7550
-	1    0    0    -1
-$EndComp
-Wire Wire Line
-	1400 7550 1400 7500
-Connection ~ 1400 7500
-Wire Wire Line
-	1400 7500 1600 7500
-Wire Wire Line
-	1400 7050 1400 7100
-Connection ~ 1400 7100
-Wire Wire Line
-	1400 7100 1600 7100
+P 1150 7550
+F 0 "#PWR0128" H 1150 7300 50  0001 C CNN
+F 1 "GND" H 1155 7377 50  0000 C CNN
+F 2 "" H 1150 7550 50  0001 C CNN
+F 3 "" H 1150 7550 50  0001 C CNN
+	1    1150 7550
+	1    0    0    -1
+$EndComp
+Wire Wire Line
+	1150 7550 1150 7500
+Wire Wire Line
+	1150 7050 1150 7100
 Text Label 10300 2600 0    50   ~ 0
 GPS_ANT
@@
 	-1   0    0    1
 $EndComp
+$Comp
+L power:+3V3 #PWR01
+U 1 1 5E25A30E
+P 9900 1550
+F 0 "#PWR01" H 9900 1400 50  0001 C CNN
+F 1 "+3V3" H 9915 1723 50  0000 C CNN
+F 2 "" H 9900 1550 50  0001 C CNN
+F 3 "" H 9900 1550 50  0001 C CNN
+	1    9900 1550
+	1    0    0    -1
+$EndComp
+Wire Wire Line
+	9450 1550 9400 1550
+Wire Wire Line
+	9900 1550 9850 1550
+Wire Wire Line
+	10500 1800 10200 1800
+Wire Wire Line
+	9650 1800 9650 1700
+Wire Wire Line
+	9650 1800 9400 1800
+Wire Wire Line
+	9400 1800 9400 1900
+Connection ~ 9650 1800
+$Comp
+L power:PWR_FLAG #FLG0104
+U 1 1 5E2D5891
+P 10200 1700
+F 0 "#FLG0104" H 10200 1775 50  0001 C CNN
+F 1 "PWR_FLAG" H 10200 1873 50  0000 C CNN
+F 2 "" H 10200 1700 50  0001 C CNN
+F 3 "~" H 10200 1700 50  0001 C CNN
+	1    10200 1700
+	1    0    0    -1
+$EndComp
+Wire Wire Line
+	10200 1700 10200 1800
+Connection ~ 10200 1800
+Wire Wire Line
+	10200 1800 9650 1800
+Wire Wire Line
+	1150 7500 1650 7500
+Wire Wire Line
+	1150 7100 1650 7100
+NoConn ~ 2150 5750
+Text Label 3600 5450 0    50   ~ 0
+MOSI
+Text Label 3600 5350 0    50   ~ 0
+MISO
+Text Label 3650 5250 0    50   ~ 0
+SCK
+Wire Wire Line
+	3350 5450 3800 5450
+Wire Wire Line
+	3350 5350 3800 5350
+Wire Wire Line
+	3350 5250 3800 5250
+$Comp
+L Jumper:SolderJumper_3_Open JP1
+U 1 1 5E5466BE
+P 9650 1550
+F 0 "JP1" H 9650 1755 50  0000 C CNN
+F 1 "backup" H 9650 1664 50  0000 C CNN
+F 2 "Jumper:SolderJumper-3_P1.3mm_Open_RoundedPad1.0x1.5mm" H 9650 1550 50  0001 C CNN
+F 3 "~" H 9650 1550 50  0001 C CNN
+	1    9650 1550
+	1    0    0    -1
+$EndComp
 $EndSCHEMATC

Commit message: Hotfixes shortly before launch
Other:
- note added: "Todo - route GPS timepulse to MCU to wake up core when fix is obtained"
Changed lines of the file:
@@
 	1    0    0    -1
 $EndComp
+Text Notes 2700 1800 0    50   ~ 0
+Todo - route GPS timepulse to MCU to wake up core when fix is obtained
 $EndSCHEMATC
