File: hw/power.sch (KiCad schematic (older format))
At the start: 31 parts, among them Q1 BC847, Q2 BC857, U6 MCP1640, U7 MCP101-270D, U8 MCP1640

Commit message: Final board
Parts:
- added J6: BAT, Connector_PinHeader_2.54mm:PinHeader_1x02_P2.54mm_Vertical, symbol Connector_Generic:Conn_01x02
- added JP2: EN, Jumper:SolderJumper-2_P1.3mm_Open_RoundedPad1.0x1.5mm, symbol Device:Jumper_NO_Small
- C18: footprint Connector_Phoenix_MC:PhoenixContact_MC_1,5_2-G-3.5_1x02_P3.50mm_Horizontal -> OptoDevice:R_LDR_5.2x5.2mm_P3.5mm_Horizontal
Connections:
- net +BATT: now also J6.2 (Pin_2), JP2.1
- net GND: now also J6.1 (Pin_1)
- net at Q2.3 (C), R17.1, R18.1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: now also JP2.2
Other:
- note added: "Common for Solar and battery power"
- note added: "Solar power, cuttable"
- moved on the sheet: C20, C21, L3, Q1, Q2, R12, R13, R14, R15, R16, R17, R18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

Commit message: Hotfixes shortly before launch
Parts:
- C20: value 100n -> 100p
Changed lines of the file:
@@
 P 10500 4300
 F 0 "C20" H 10615 4346 50  0000 L CNN
-F 1 "100n" H 10615 4255 50  0000 L CNN
+F 1 "100p" H 10615 4255 50  0000 L CNN
 F 2 "Capacitor_SMD:C_0603_1608Metric" H 10538 4150 50  0001 C CNN
 F 3 "~" H 10500 4300 50  0001 C CNN
